File: Raspi-On-Off_PMos_SMD_nl.sch (EAGLE design)
At the start: 32 parts, among them IC1 74AUC1G17, T1 FDC6327C, T2 FDC6327C, T3 BSS123, T4 IRF7416, T5 IRLML0030, X1 MKDSN1,5/2-5,08

Commit message: Add files via upload
Parts:
- T3: value BSS123 -> IRLML2803
Changed lines of the file:
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@@
 <part name="GND5" library="supply1" deviceset="GND" device=""/>
 <part name="R3" library="rcl" deviceset="R-EU_" device="R0805" value="270R"/>
-<part name="T3" library="transistor-small-signal" deviceset="BSS123" device="23" value="BSS123"/>
+<part name="T3" library="transistor-small-signal" deviceset="BSS123" device="23" value="IRLML2803"/>
 <part name="LED2" library="led" deviceset="LED" device="3MM" value="red"/>
 <part name="T5" library="transistor-small-signal" deviceset="BSS123" device="23" value="IRLML0030"/>
